File: agentosaurus/cm4-slot.kicad_sch (KiCad schematic)
At the start: 13 parts, among them J1 DF40HC-100DS, J2 DF40HC-100DS, J3 M2_Key_M_NVMe, J4 MicroSD_Card_Slot, T1 HX1188NL

Commit message: Fix M.2 floating pins (CLKREQ#, PEWAKE#) and rewrite README for Agentosaurus
Add 10k pull-up resistors to VCC3V3 on J3 CLKREQ# (pin 12) and PEWAKE#
(pin 19) in cm4-slot.kicad_sch. These PCIe power management inputs were
floating, which can cause SSD link training failures or unpredictable
wake behavior. Pull-ups keep clock always-on and disable wake signaling,
appropriate for an always-on embedded system.

Rewrite README.md to describe Agentosaurus (4-node CM4/CM5 cluster board,
Mini-ITX, RTL8367S switch, ESP32-S3 BMC) instead of the original single-node
Antmicro Scalenode.

Co-Authored-By: Claude Opus 4.6 (1M context) <noreply@anthropic.com>
Parts:
- added R1, R2: 10k, Resistor_SMD:R_0402_1005Metric, symbol Device:R
Other:
- note added: "M.2 PCIe Pull-Ups"
Changed lines of the file:
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@@
+  )
+  ;; ===============================================================
+  ;; CLKREQ# and PEWAKE# Pull-Up Resistors (10k to VCC3V3)
+  ;; ===============================================================
+  (text "M.2 PCIe Pull-Ups" (at 63.5 229.0 0)
+    (effects (font (size 1.27 1.27) bold) (justify left bottom))
+  )
+  ;; R1 — 10k pull-up on CLKREQ# (J3 pin 12, right side at 53.34, 241.3)
+  ;; Wire from J3 pin 12 to resistor
+  (wire (pts (xy 53.34 241.3) (xy 63.5 241.3))
+    (stroke (width 0) (type default))
+  )
+  ;; R1 at (63.5, 237.49) — pin 2 bottom at 241.3, pin 1 top at 233.68
+  (symbol (lib_id "Device:R") (at 63.5 237.49 0) (unit 1)
+    (in_bom yes) (on_board yes)
+    (property "Reference" "R1" (at 66.04 237.49 0) (effects (font (size 1.27 1.27)) (justify left)))
+    (property "Value" "10k" (at 66.04 239.49 0) (effects (font (size 1.27 1.27)) (justify left)))
+    (property "Footprint" "Resistor_SMD:R_0402_1005Metric" (at 65.278 237.49 90) (effects (font (size 1.27 1.27)) hide))
+    (property "Datasheet" "" (at 63.5 237.49 0) (effects (font (size 1.27 1.27)) hide))
+    (instances (project "agentosaurus" (path "/c1000001-0001-4000-8000-000000000001" (reference "R1") (unit 1))))
+  )
+  ;; VCC3V3 power symbol for R1 top
+  (symbol (lib_id "power:VCC3V3") (at 63.5 233.68 0) (unit 1)
+    (in_bom yes) (on_board yes)
+    (property "Reference" "#PWR027" (at 63.5 237.49 0) (effects (font (size 1.27 1.27)) hide))
+    (property "Value" "VCC3V3" (at 63.5 231.14 0) (effects (font (size 1.27 1.27))))
+    (property "Footprint" "" (at 63.5 233.68 0) (effects (font (size 1.27 1.27)) hide))
+    (property "Datasheet" "" (at 63.5 233.68 0) (effects (font (size 1.27 1.27)) hide))
+    (instances (project "agentosaurus" (path "/c1000001-0001-4000-8000-000000000001" (reference "#PWR027") (unit 1))))
+  )
+  ;; R2 — 10k pull-up on PEWAKE# (J3 pin 19, left side at 22.86, 231.14)
+  ;; Wire from J3 pin 19 to resistor
+  (wire (pts (xy 22.86 231.14) (xy 12.7 231.14))
+    (stroke (width 0) (type default))
+  )
+  ;; R2 at (12.7, 227.33) — pin 2 bottom at 231.14, pin 1 top at 223.52
+  (symbol (lib_id "Device:R") (at 12.7 227.33 0) (unit 1)
+    (in_bom yes) (on_board yes)
+    (property "Reference" "R2" (at 15.24 227.33 0) (effects (font (size 1.27 1.27)) (justify left)))
+    (property "Value" "10k" (at 15.24 229.33 0) (effects (font (size 1.27 1.27)) (justify left)))
+    (property "Footprint" "Resistor_SMD:R_0402_1005Metric" (at 14.478 227.33 90) (effects (font (size 1.27 1.27)) hide))
+    (property "Datasheet" "" (at 12.7 227.33 0) (effects (font (size 1.27 1.27)) hide))
+    (instances (project "agentosaurus" (path "/c1000001-0001-4000-8000-000000000001" (reference "R2") (unit 1))))
+  )
+  ;; VCC3V3 power symbol for R2 top
+  (symbol (lib_id "power:VCC3V3") (at 12.7 223.52 0) (unit 1)
+    (in_bom yes) (on_board yes)
+    (property "Reference" "#PWR028" (at 12.7 227.33 0) (effects (font (size 1.27 1.27)) hide))
+    (property "Value" "VCC3V3" (at 12.7 220.98 0) (effects (font (size 1.27 1.27))))
+    (property "Footprint" "" (at 12.7 223.52 0) (effects (font (size 1.27 1.27)) hide))
+    (property "Datasheet" "" (at 12.7 223.52 0) (effects (font (size 1.27 1.27)) hide))
+    (instances (project "agentosaurus" (path "/c1000001-0001-4000-8000-000000000001" (reference "#PWR028") (unit 1))))
   )
   ;; ===============================================================
